Commit message: Add robot description files and launch configuration for Gazebo simulation
- Included gazebo_control.xacro for simulation plugins
- Updated robot.urdf.xacro to include gazebo_control.xacro
- Created gz_bridge.yaml for ROS-Gazebo topic bridging
- Added view_robot.rviz for visualization settings
- Implemented launch_sim.launch.py to orchestrate simulation launch

File: description/robot_core.xacro (robot description, xacro)
@@ -14,8 +14,7 @@
         <color rgba="0 0 0 1"/>
     </material>
-    <!-- BASE LINK -->
     <link name="base_link">
     </link>
-    <!-- CHASSIS LINK -->
+    <!-- Chassis -->
     <joint name="chassis_joint" type="fixed">
         <parent link="base_link"/>
@@ -25,5 +24,5 @@
     <link name="chassis">
         <visual>
-            <origin xyz="0.15 0 0.075"/>
+            <origin xyz="0.15 0 0.075" rpy="0 0 0"/>
             <geometry>
                 <box size="0.3 0.3 0.15"/>
@@ -32,5 +31,5 @@
         </visual>
         <collision>
-            <origin xyz="0.15 0 0.075"/>
+            <origin xyz="0.15 0 0.075" rpy="0 0 0"/>
             <geometry>
                 <box size="0.3 0.3 0.15"/>
@@ -41,5 +40,5 @@
         </xacro:inertial_box>
     </link>
-    <!-- LEFT WHEEL LINK -->
+    <!-- LEFT WHEEL -->
     <joint name="left_wheel_joint" type="continuous">
         <parent link="base_link"/>
@@ -47,9 +46,10 @@
         <origin xyz="0 0.175 0" rpy="-${pi/2} 0 0"/>
         <axis xyz="0 0 1"/>
+        <limit effort="0.05" velocity="10.0"/>
     </joint>
     <link name="left_wheel">
         <visual>
             <geometry>
-                <cylinder radius="0.05" length="0.04"/>
+                <cylinder length="0.04" radius="0.05" />
             </geometry>
             <material name="blue"/>
@@ -57,5 +57,5 @@
         <collision>
             <geometry>
-                <cylinder radius="0.05" length="0.04"/>
+                <sphere radius="0.05" />
             </geometry>
         </collision>
@@ -64,5 +64,5 @@
         </xacro:inertial_cylinder>
     </link>
-    <!-- RIGHT WHEEL LINK -->
+    <!-- RIGHT WHEEL -->
     <joint name="right_wheel_joint" type="continuous">
         <parent link="base_link"/>
@@ -70,9 +70,10 @@
         <origin xyz="0 -0.175 0" rpy="${pi/2} 0 0"/>
         <axis xyz="0 0 -1"/>
+        <limit effort="0.05" velocity="10.0"/>
     </joint>
     <link name="right_wheel">
         <visual>
             <geometry>
-                <cylinder radius="0.05" length="0.04"/>
+                <cylinder length="0.04" radius="0.05" />
             </geometry>
             <material name="blue"/>
@@ -80,5 +81,5 @@
         <collision>
             <geometry>
-                <cylinder radius="0.05" length="0.04"/>
+                <sphere radius="0.05" />
             </geometry>
         </collision>
@@ -87,14 +88,14 @@
         </xacro:inertial_cylinder>
     </link>
-    <!-- CASTOR WHEEL LINK -->
-    <joint name="castor_wheel_joint" type="fixed">
+    <!-- CASTER WHEEL -->
+    <joint name="caster_wheel_joint" type="fixed">
         <parent link="chassis"/>
-        <child link="castor_wheel"/>
-        <origin xyz="0.24 0 0"/>
+        <child link="caster_wheel"/>
+        <origin xyz="0.24 0 0" rpy="0 0 0"/>
     </joint>
-    <link name="castor_wheel">
+    <link name="caster_wheel">
         <visual>
             <geometry>
-                <sphere radius="0.05"/>
+                <sphere radius="0.05" />
             </geometry>
             <material name="black"/>
@@ -102,10 +103,14 @@
         <collision>
             <geometry>
-                <sphere radius="0.05"/>
+                <sphere radius="0.05" />
             </geometry>
         </collision>
-        <xacro:inertial_sphere mass="0.05" radius="0.05">
+        <xacro:inertial_sphere mass="0.1" radius="0.05">
             <origin xyz="0 0 0" rpy="0 0 0"/>
         </xacro:inertial_sphere>
     </link>
+    <gazebo reference="caster_wheel">
+        <mu1 value="0.0"/>
+        <mu2 value="0.0"/>
+    </gazebo>
 </robot>

Commit message: Add base footprint joint and link to robot description; introduce mapper parameters for SLAM configuration

File: description/robot_core.xacro (robot description, xacro)
@@ -36,4 +36,12 @@
     <!-- BASE LINK -->
     <link name="base_link">
+    </link>
+    <!-- BASE_FOOTPRINT -->
+    <joint name="base_footprint_joint" type="fixed">
+        <parent link="base_link"/>
+        <child link="base_footprint"/>
+        <origin xyz="0 0 0" rpy="0 0 0"/>
+    </joint>
+    <link name="base_footprint">
     </link>
     <!-- CHASSIS LINK -->
